File: Hardware/SegmentTestBoard/SegmentTestBoard.kicad_sch (KiCad schematic)
At the start: 13 parts, among them J101 OUT, J102 IN, U101 SN74HC595, U102 STATE

Commit message: use correct pinheaders
Parts:
- J101, J102: footprint Connector_PinHeader_1.00mm:PinHeader_1x05_P1.00mm_Vertical -> Connector_PinHeader_2.54mm:PinHeader_1x05_P2.54mm_Vertical
Changed lines of the file:
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@@
       (effects (font (size 1.27 1.27)) (justify right))
     )
-    (property "Footprint" "Connector_PinHeader_1.00mm:PinHeader_1x05_P1.00mm_Vertical" (at 77.47 143.51 0)
+    (property "Footprint" "Connector_PinHeader_2.54mm:PinHeader_1x05_P2.54mm_Vertical" (at 77.47 143.51 0)
       (effects (font (size 1.27 1.27)) hide)
     )
@@
       (effects (font (size 1.27 1.27)) (justify right))
     )
-    (property "Footprint" "Connector_PinHeader_1.00mm:PinHeader_1x05_P1.00mm_Vertical" (at 77.47 116.205 0)
-      (effects (font (size 1.27 1.27)) hide)
-    )
+    (property "Footprint" "Connector_PinHeader_2.54mm:PinHeader_1x05_P2.54mm_Vertical" (at 77.47 116.205 0)
+      (effects (font (size 1.27 1.27)) hide)
+    )

Commit message: Add final bits
Other:
- company: (none) -> Kitsune Robotics
- title: (none) -> Segment Test Board
Changed lines of the file:
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@@
 (kicad_sch (version 20230121) (generator eeschema)
   (paper "A4")
+  (title_block
+    (title "Segment Test Board")
+    (date "${ISSUE}")
+    (rev "${REVISION}")
+    (company "Kitsune Robotics")
+    (comment 5 "${FULL_REVISION}")
+  )
   (junction (at 207.01 127.635) (diameter 0) (color 0 0 0 0)
   )
